File: alien.sch (KiCad schematic (older format))
At the start: 26 parts

Commit message: solo falta el amplificador de audio
Parts:
- added C?: 0.001uF, symbol C
- added C?: 100pF, symbol C
- added D?: D, symbol D
- added Q?: 2N5457, symbol Q_NJFET_GDS
- added R?: 2M, symbol R
- added R? (x3): 10k, symbol R
- added R?: 100k, symbol R
- added R?: 300k, symbol R
- added R?: 15k, symbol R
- added SW?: SW_SPST, symbol SW_SPST
- added U? (x2): LM324, symbol LM324
- Q? (x2): value NPN -> 2N3904
Connections:
- net +9VA: now also R?.2, U?.4 (V+)
- net -9VA: now also R?.1, R?.1, R?.2, U?.11 (V-)
- net GNDREF: now also U?.3 (+)
- net at C?.2, R?.1, R?.1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: now also SW?.1 (A)
- net at Q?.2 (C): now also C?.2, Q?.3 (S), U?.2 (-)
- new net: C?.1, Q?.2 (D), R?.1, U?.1
- new net: Q?.1 (G), R?.1, R?.2
- new net: D?.1 (K), R?.2
- new net: C?.2, R?.1, SW?.2 (B)
- new net: C?.1, R?.1, R?.2, U?.6 (-)
- new net: R?.1, R?.2, U?.5 (+)
- new net: D?.2 (A), R?.2, U?.7

Commit message: alimentación
Parts:
- added BT?: 9 V battery, symbol Battery_Cell
- added C?: 470uF, symbol CP1
- added C? (x2): 0.1uF, symbol C
- added R? (x2): 4k7, symbol R
- added SW?: SW_SPST, symbol SW_SPST
Connections:
- net +9VA: now also C?.1, C?.2, R?.1, SW?.2 (B)
- net -9VA: now also BT?.2 (-), C?.1, C?.2, R?.2
- net GNDREF: now also C?.1, C?.2, R?.1, R?.2
- new net: BT?.1 (+), SW?.1 (A)
Changed lines of the file:
@@
 	-1   0    0    1
+$EndComp
+$Comp
+L Battery_Cell BT?
+U 1 1 5935E30E
+P 1200 5450
+F 0 "BT?" H 1300 5550 50  0000 L CNN
+F 1 "9 V battery" H 750 5400 50  0000 L CNN
+F 2 "" V 1200 5510 50  0001 C CNN
+F 3 "" V 1200 5510 50  0001 C CNN
+	1    1200 5450
+	1    0    0    -1
+$EndComp
+$Comp
+L SW_SPST SW?
+U 1 1 5935EA4D
+P 1500 4900
+F 0 "SW?" H 1500 5025 50  0000 C CNN
+F 1 "SW_SPST" H 1500 4800 50  0000 C CNN
+F 2 "" H 1500 4900 50  0001 C CNN
+F 3 "" H 1500 4900 50  0001 C CNN
+	1    1500 4900
+	1    0    0    -1
+$EndComp
+$Comp
+L CP1 C?
+U 1 1 5935EE03
+P 1700 5400
+F 0 "C?" H 1725 5500 50  0000 L CNN
+F 1 "470uF" H 1725 5300 50  0000 L CNN
+F 2 "" H 1700 5400 50  0001 C CNN
+F 3 "" H 1700 5400 50  0001 C CNN
+	1    1700 5400
+	1    0    0    -1
+$EndComp
+$Comp
+L R R?
+U 1 1 5935F338
+P 2100 5200
+F 0 "R?" V 2180 5200 50  0000 C CNN
+F 1 "4k7" V 2100 5200 50  0000 C CNN
+F 2 "" V 2030 5200 50  0001 C CNN
+F 3 "" H 2100 5200 50  0001 C CNN
+	1    2100 5200
+	1    0    0    -1
+$EndComp
+$Comp
+L R R?
+U 1 1 5935F418
+P 2100 5600
+F 0 "R?" V 2180 5600 50  0000 C CNN
+F 1 "4k7" V 2100 5600 50  0000 C CNN
+F 2 "" V 2030 5600 50  0001 C CNN
+F 3 "" H 2100 5600 50  0001 C CNN
+	1    2100 5600
+	1    0    0    -1
+$EndComp
+$Comp
+L GNDREF #PWR?
+U 1 1 5935F631
+P 2400 5450
+F 0 "#PWR?" H 2400 5200 50  0001 C CNN
+F 1 "GNDREF" H 2400 5300 50  0000 C CNN
+F 2 "" H 2400 5450 50  0001 C CNN
+F 3 "" H 2400 5450 50  0001 C CNN
+	1    2400 5450
+	1    0    0    -1
 $EndComp
 Wire Wire Line
@@
 Wire Wire Line
 	2050 3500 6400 3500
+Wire Wire Line
+	1200 5250 1200 4900
+Wire Wire Line
+	1200 4900 1300 4900
+Wire Wire Line
+	1700 4900 2100 4900
+Wire Wire Line
+	2100 4900 2100 5050
+Wire Wire Line
+	2100 5350 2100 5450
+Wire Wire Line
+	2100 5400 2400 5400
+Wire Wire Line
+	2400 5400 2400 5450
+Connection ~ 2100 5400
+Wire Wire Line
+	1200 5550 1200 5950
+Wire Wire Line
+	1200 5950 2100 5950
+Wire Wire Line
+	2100 5950 2100 5750
+Connection ~ 1700 5950
+Connection ~ 1700 4900
+Wire Wire Line
+	1700 4750 1700 5250
+Wire Wire Line
+	1700 5550 1700 6100
+$Comp
+L -9VA #PWR?
+U 1 1 5936112D
+P 1700 6100
+F 0 "#PWR?" H 1700 5975 50  0001 C CNN
+F 1 "-9VA" H 1700 6250 50  0000 C CNN
+F 2 "" H 1700 6100 50  0001 C CNN
+F 3 "" H 1700 6100 50  0001 C CNN
+	1    1700 6100
+	-1   0    0    1
+$EndComp
+$Comp
+L +9VA #PWR?
+U 1 1 5936148F
+P 1700 4750
+F 0 "#PWR?" H 1700 4625 50  0001 C CNN
+F 1 "+9VA" H 1700 4900 50  0000 C CNN
+F 2 "" H 1700 4750 50  0001 C CNN
+F 3 "" H 1700 4750 50  0001 C CNN
+	1    1700 4750
+	1    0    0    -1
+$EndComp
+$Comp
+L PWR_FLAG #FLG?
+U 1 1 59361906
+P 2050 4750
+F 0 "#FLG?" H 2050 4825 50  0001 C CNN
+F 1 "PWR_FLAG" H 2050 4900 50  0000 C CNN
+F 2 "" H 2050 4750 50  0001 C CNN
+F 3 "" H 2050 4750 50  0001 C CNN
+	1    2050 4750
+	1    0    0    -1
+$EndComp
+$Comp
+L PWR_FLAG #FLG?
+U 1 1 593619CC
+P 2050 6100
+F 0 "#FLG?" H 2050 6175 50  0001 C CNN
+F 1 "PWR_FLAG" H 2050 6250 50  0000 C CNN
+F 2 "" H 2050 6100 50  0001 C CNN
+F 3 "" H 2050 6100 50  0001 C CNN
+	1    2050 6100
+	-1   0    0    1
+$EndComp
+Wire Wire Line
+	2050 4750 2050 4900
+Connection ~ 2050 4900
+Wire Wire Line
+	2050 6100 2050 5950
+Connection ~ 2050 5950
+$Comp
+L C C?
+U 1 1 59362971
+P 3150 5150
+F 0 "C?" H 3175 5250 50  0000 L CNN
+F 1 "0.1uF" H 3175 5050 50  0000 L CNN
+F 2 "" H 3188 5000 50  0001 C CNN
+F 3 "" H 3150 5150 50  0001 C CNN
+	1    3150 5150
+	-1   0    0    1
+$EndComp
+$Comp
+L C C?
+U 1 1 59362E97
+P 3150 5650
+F 0 "C?" H 3175 5750 50  0000 L CNN
+F 1 "0.1uF" H 3175 5550 50  0000 L CNN
+F 2 "" H 3188 5500 50  0001 C CNN
+F 3 "" H 3150 5650 50  0001 C CNN
+	1    3150 5650
+	-1   0    0    1
+$EndComp
+$Comp
+L GNDREF #PWR?
+U 1 1 59362F48
+P 3400 5450
+F 0 "#PWR?" H 3400 5200 50  0001 C CNN
+F 1 "GNDREF" H 3400 5300 50  0000 C CNN
+F 2 "" H 3400 5450 50  0001 C CNN
+F 3 "" H 3400 5450 50  0001 C CNN
+	1    3400 5450
+	1    0    0    -1
+$EndComp
+Wire Wire Line
+	3150 5300 3150 5500
+Wire Wire Line
+	3150 5400 3400 5400
+Wire Wire Line
+	3400 5400 3400 5450
+Connection ~ 3150 5400
+$Comp
+L -9VA #PWR?
+U 1 1 59363141
+P 3150 5900
+F 0 "#PWR?" H 3150 5775 50  0001 C CNN
+F 1 "-9VA" H 3150 6050 50  0000 C CNN
+F 2 "" H 3150 5900 50  0001 C CNN
+F 3 "" H 3150 5900 50  0001 C CNN
+	1    3150 5900
+	-1   0    0    1
+$EndComp
+$Comp
+L +9VA #PWR?
+U 1 1 593631D9
+P 3150 4950
+F 0 "#PWR?" H 3150 4825 50  0001 C CNN
+F 1 "+9VA" H 3150 5100 50  0000 C CNN
+F 2 "" H 3150 4950 50  0001 C CNN
+F 3 "" H 3150 4950 50  0001 C CNN
+	1    3150 4950
+	1    0    0    -1
+$EndComp
+Wire Wire Line
+	3150 5000 3150 4950
+Wire Wire Line
+	3150 5900 3150 5800
 $EndSCHEMATC

Commit message: erc ok
Parts:
- added C10: 1uF, symbol C
- added J1: Audio-Jack-2, symbol Audio-Jack-2
- added R22: 100k, symbol R
- added R23: 4k7, symbol R
- added RV4: 100k, symbol POT
- gave numbers to parts that had none: 44
Connections:
- net -9VA: now also R23.1, RV4.3
- net GNDREF: now also U1.10 (+), U1.5 (+), J1.2; no longer U1.12 (+), U1.3 (+)
- net at R1.2, R2.1, R4.2: now also U1.3 (+); no longer U1.10 (+)
- net at C3.2, R4.1, R5.1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: now also U1.1; no longer U1.8
- net at C1.1, R3.2: now also U1.2 (-)
- net at C7.2, Q1.2 (C), R13.1: now also U1.6 (-); no longer U1.13 (-)
- net at C7.1, R14.1: now also U1.7; no longer U1.14
- net at C8.2, Q2.2 (C), Q3.3 (S): now also U1.9 (-); no longer U1.2 (-)
- net at C8.1, Q3.2 (D), R18.1: now also U1.8, RV4.1; no longer U1.1
- net at C9.1, R16.1, R17.2: now also U1.13 (-); no longer U1.6 (-)
- net at R18.2, R19.1: now also U1.12 (+); no longer U1.5 (+)
- net at D2.2 (A), R19.2: now also U1.14; no longer U1.7
- new net: C10.1, J1.1, R22.2
- new net: C10.2, RV4.2
- new net: R22.1, R23.2
Other:
- moved on the sheet: C5, D2, R20, R21, R3
