File: alien.sch (KiCad schematic (older format))
At the start: 49 parts, among them J1 Audio-Jack-2, Q1 2N3904, Q2 2N3904, Q3 2N5457, SW1 SW_SPST, SW2 SW_SPST, SW3 SW_SPDT, SW4 SW_SPST, U1 LM324

Commit message: conectores para panel
Parts:
- removed R23: 4k7, symbol R
- added X1, X2, X3, X4, X5, X6, X7, X8: JD_CONN_01X01, symbol JD_CONN_01X01
- R22: value 100k -> 150k
Connections:
- net -9VA: now also R22.1
- net at C3.2, R4.1, R5.1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: now also X3.1
- net at R3.1, RV1.1: now also X1.1
- net at D1.2 (A), R5.2: now also X2.1
- net at C4.1, R8.1, SW3.3 (C): now also X4.1
- net at Q1.1 (B), R10.1, R11.2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: now also X6.1
- net at R10.2, RV3.2: now also X5.1
- net at C10.1, J1.1, R22.2: now also X8.1
- net at C10.2, RV4.2: now also X7.1
Other:
- moved on the sheet: BT1, C1, C10, C2, C3, C4, C5, C6, C7, C8, C9, D1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

Commit message: comenzando a asignar huellas
Parts:
- U1: footprint (none) -> Housings_DIP:DIP-14_W7.62mm_LongPads
- X1, X2, X3, X4, X5, X6, X7, X8: footprint (none) -> Mounting_Holes:MountingHole_2.5mm_Pad
Changed lines of the file:
@@
 F 0 "U1" H 1600 2500 50  0000 L CNN
 F 1 "LM324" H 1600 2100 50  0000 L CNN
-F 2 "" H 1550 2400 50  0001 C CNN
+F 2 "Housings_DIP:DIP-14_W7.62mm_LongPads" H 1550 2400 50  0001 C CNN
 F 3 "" H 1650 2500 50  0001 C CNN
 	3    1600 2300
@@
 F 0 "U1" H 5450 3850 50  0000 L CNN
 F 1 "LM324" H 5450 3450 50  0000 L CNN
-F 2 "" H 5400 3750 50  0001 C CNN
+F 2 "Housings_DIP:DIP-14_W7.62mm_LongPads" H 5400 3750 50  0001 C CNN
 F 3 "" H 5500 3850 50  0001 C CNN
 	4    5450 3650
@@
 F 0 "U1" H 7250 2150 50  0000 L CNN
 F 1 "LM324" H 7250 1750 50  0000 L CNN
-F 2 "" H 7200 2050 50  0001 C CNN
+F 2 "Housings_DIP:DIP-14_W7.62mm_LongPads" H 7200 2050 50  0001 C CNN
 F 3 "" H 7300 2150 50  0001 C CNN
 	1    7250 1950
@@
 F 0 "U1" H 8500 2900 50  0000 L CNN
 F 1 "LM324" H 8500 2500 50  0000 L CNN
-F 2 "" H 8450 2800 50  0001 C CNN
+F 2 "Housings_DIP:DIP-14_W7.62mm_LongPads" H 8450 2800 50  0001 C CNN
 F 3 "" H 8550 2900 50  0001 C CNN
 	2    8500 2700
@@
 F 0 "X1" H 1700 1350 50  0000 C CNN
 F 1 "JD_CONN_01X01" H 1550 1250 50  0001 C CNN
-F 2 "" H 1550 1350 50  0001 C CNN
+F 2 "Mounting_Holes:MountingHole_2.5mm_Pad" H 1550 1350 50  0001 C CNN
 F 3 "" H 1550 1350 50  0001 C CNN
 	1    1550 1350
@@
 F 0 "X3" H 2250 1850 50  0000 C CNN
 F 1 "JD_CONN_01X01" H 2100 1750 50  0001 C CNN
-F 2 "" H 2100 1850 50  0001 C CNN
+F 2 "Mounting_Holes:MountingHole_2.5mm_Pad" H 2100 1850 50  0001 C CNN
 F 3 "" H 2100 1850 50  0001 C CNN
 	1    2100 1850
@@
 F 0 "X4" H 3100 2950 50  0000 C CNN
 F 1 "JD_CONN_01X01" H 2950 2850 50  0001 C CNN
-F 2 "" H 2950 2950 50  0001 C CNN
+F 2 "Mounting_Holes:MountingHole_2.5mm_Pad" H 2950 2950 50  0001 C CNN
 F 3 "" H 2950 2950 50  0001 C CNN
 	1    2950 2950
@@
 F 0 "X6" H 4650 1800 50  0000 C CNN
 F 1 "JD_CONN_01X01" H 4500 1700 50  0001 C CNN
-F 2 "" H 4500 1800 50  0001 C CNN
+F 2 "Mounting_Holes:MountingHole_2.5mm_Pad" H 4500 1800 50  0001 C CNN
 F 3 "" H 4500 1800 50  0001 C CNN
 	1    4500 1800
@@
 F 0 "X5" H 4000 3250 50  0000 C CNN
 F 1 "JD_CONN_01X01" H 3850 3150 50  0001 C CNN
-F 2 "" H 3850 3250 50  0001 C CNN
+F 2 "Mounting_Holes:MountingHole_2.5mm_Pad" H 3850 3250 50  0001 C CNN
 F 3 "" H 3850 3250 50  0001 C CNN
 	1    3850 3250
@@
 F 0 "X2" H 1850 3450 50  0000 C CNN
 F 1 "JD_CONN_01X01" H 1700 3350 50  0001 C CNN
-F 2 "" H 1700 3450 50  0001 C CNN
+F 2 "Mounting_Holes:MountingHole_2.5mm_Pad" H 1700 3450 50  0001 C CNN
 F 3 "" H 1700 3450 50  0001 C CNN
 	1    1700 3450
@@
 F 0 "X7" H 9900 1900 50  0000 C CNN
 F 1 "JD_CONN_01X01" H 9750 1800 50  0001 C CNN
-F 2 "" H 9750 1900 50  0001 C CNN
+F 2 "Mounting_Holes:MountingHole_2.5mm_Pad" H 9750 1900 50  0001 C CNN
 F 3 "" H 9750 1900 50  0001 C CNN
 	1    9750 1900
@@
 F 0 "X8" H 10500 1900 50  0000 C CNN
 F 1 "JD_CONN_01X01" H 10350 1800 50  0001 C CNN
-F 2 "" H 10350 1900 50  0001 C CNN
+F 2 "Mounting_Holes:MountingHole_2.5mm_Pad" H 10350 1900 50  0001 C CNN
 F 3 "" H 10350 1900 50  0001 C CNN
 	1    10350 1900

Commit message: casi para enrutar
Parts:
- removed J1: Audio-Jack-2, symbol Audio-Jack-2
- added J1: Jack_3.5mm_2pin, symbol Jack_3.5mm_2pin
- added X10, X11, X9: JD_CONN_01X01, Mounting_Holes:MountingHole_2.5mm_Pad, symbol JD_CONN_01X01
- added X12, X13: JD_CONN_01X02, Connectors:bornier2, symbol JD_CONN_01X02
- C1, C10, C3, C4: footprint (none) -> Capacitors_THT:CP_Radial_D5.0mm_P2.50mm
- C2: footprint (none) -> Capacitors_THT:CP_Radial_D12.5mm_P5.00mm
- C5, C6, C7, C8, C9: footprint (none) -> Capacitors_THT:C_Disc_D5.0mm_W2.5mm_P5.00mm
- D1: footprint (none) -> LEDs:LED_D5.0mm
- D2: footprint (none) -> Diodes_THT:D_DO-35_SOD27_P7.62mm_Horizontal
- Q1, Q2, Q3: footprint (none) -> TO_SOT_Packages_THT:TO-92_Inline_Wide
- R1, R10, R11, R12, R13, R14, R15, R16, R17, R18, R19, R2, R20, R21, R22, R3, R4, R5, R6, R7, R8, R9: footprint (none) -> Resistors_THT:R_Axial_DIN0207_L6.3mm_D2.5mm_P7.62mm_Horizontal
Connections:
- wire segments 118 -> 124
Other:
- moved on the sheet: R6, R7, X6

Commit message: corrección de la posición de las patas de los transistores
Parts:
- removed Q1, Q2: 2N3904, TO_SOT_Packages_THT:TO-92_Inline_Wide, symbol Q_NPN_BCE
- removed Q3: 2N5457, TO_SOT_Packages_THT:TO-92_Inline_Wide, symbol Q_NJFET_GDS
- added Q1, Q2: 2N390, TO_SOT_Packages_THT:TO-92_Inline_Wide, symbol BC237
- added Q3: 2N5457, TO_SOT_Packages_THT:TO-92_Inline_Wide, symbol BF245A
- C9: value 100pF -> 0.01
