File: _saved_alien.sch (KiCad schematic (older format))
At the start: 56 parts, among them J1 Audio-Jack-2, Q1 2N3904, Q2 2N3904, Q3 2N5457, SW1 SW_SPST, SW2 SW_SPST, SW3 SW_SPDT, SW4 SW_SPST, U1 LM324, X1 JD_CONN_01X01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

Commit message: casi para enrutar
Parts:
- removed J1: Audio-Jack-2, symbol Audio-Jack-2
- added J1: Jack_3.5mm_2pin, symbol Jack_3.5mm_2pin
- added X10, X11, X9: JD_CONN_01X01, Mounting_Holes:MountingHole_2.5mm_Pad, symbol JD_CONN_01X01
- added X12, X13: JD_CONN_01X02, Connectors:bornier2, symbol JD_CONN_01X02
- R1, R10, R11, R12, R13, R15, R16, R17, R18, R19, R2, R20, R21, R22, R3, R4, R5, R6, R7, R8, R9: footprint (none) -> Resistors_THT:R_Axial_DIN0207_L6.3mm_D2.5mm_P7.62mm_Horizontal
- R14: footprint (none) -> Resistors_THT:R_Axial_DIN0204_L3.6mm_D1.6mm_P1.90mm_Vertical
Connections:
- wire segments 118 -> 124
Other:
- moved on the sheet: R6, R7, X6
