File: alien.kicad_pcb (KiCad board)
At the start: 2 copper layers, 49 parts, among them Q1 2N3904, Q2 2N3904, Q3 2N5457, U1 LM324, X1 JD_CONN_01X01, X10 JD_CONN_01X01, X11 JD_CONN_01X01, X12 JD_CONN_01X02, X13 JD_CONN_01X02, X2 JD_CONN_01X01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

Commit message: empezamos a enrutar
Parts:
- added REF**: 1pin, Connectors:1pin, F.Cu at (138.0, 144.0)
- added REF**: 1pin, Connectors:1pin, F.Cu at (76.0, 68.0)
- moved X11 32.1 mm to (85.0, 69.0)
- moved X2 18.0 mm to (84.7, 143.0)
- moved X10 13.6 mm to (111.0, 69.0)
- moved R7 10.5 mm to (96.0, 80.0), turned to 0 degrees
- moved X3 8.78 mm to (92.4, 143.0)
- moved X4 8.44 mm to (100.1, 143.0)
- moved X6 8.26 mm to (107.9, 143.0)
- moved X5 7.97 mm to (115.6, 143.0)
- moved X7 7.49 mm to (123.3, 143.0)
- moved X8 7.20 mm to (131.0, 143.0)
- moved X9 4.90 mm to (137.0, 69.0)
- moved R3 4.65 mm to (77.0, 130.8)
- moved R5 4.65 mm to (80.5, 130.8)
- moved R18 4.11 mm to (139.0, 88.5), turned to 180 degrees
- moved R21 4.10 mm to (139.0, 80.5), turned to 180 degrees
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Other:
- board outline added: 70 x 84 mm
- net class sinte added: clearance 0.5, trace_width 0.8, via_dia 0.6, via_drill 0.4

Commit message: primera versión con autorouting
Parts:
- moved X8 2.00 mm to (129.0, 143.0)
- moved X7 1.71 mm to (121.6, 143.0)
- moved X5 1.43 mm to (114.1, 143.0)
- moved X6 1.14 mm to (106.7, 143.0)
- moved X4 0.86 mm to (99.3, 143.0)
- moved X3 0.57 mm to (91.9, 143.0)
- moved X2 0.29 mm to (84.4, 143.0)
Routing:
- net -9VA: track 0.00 -> 191.1 mm, vias 0 -> 3
- net +9VA: track 0.00 -> 133.6 mm
- net GNDREF: track 0.00 -> 120.6 mm, vias 0 -> 3
- net Net-(C7-Pad2): track 0.00 -> 67.8 mm, vias 0 -> 3
- net Net-(C8-Pad1): track 0.00 -> 67.8 mm, vias 0 -> 1
- net Net-(C3-Pad2): track 0.00 -> 59.1 mm, vias 0 -> 2
- net Net-(C8-Pad2): track 0.00 -> 44.2 mm, vias 0 -> 2
- net Net-(D2-Pad2): track 0.00 -> 38.6 mm, vias 0 -> 2
- net Net-(R18-Pad2): track 0.00 -> 37.0 mm, vias 0 -> 2
- net Net-(R1-Pad2): track 0.00 -> 34.4 mm
- net Net-(Q1-Pad3): track 0.00 -> 34.0 mm
- net Net-(C9-Pad1): track 0.00 -> 33.5 mm
- net Net-(C4-Pad1): track 0.00 -> 33.4 mm
- net Net-(C1-Pad1): track 0.00 -> 32.8 mm, vias 0 -> 1
- net Net-(Q3-Pad1): track 0.00 -> 29.9 mm
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Other:
- net class Default: clearance 0.2 -> 0.5; trace_width 0.25 -> 0.8
- rule trace_clearance: 0.2 -> 0.5
- rule trace_min: 0.2 -> 0.5

Commit message: amo que nos vamos
Parts:
- moved X1 110.5 mm to (185.2, 120.6), turned to 90 degrees
- moved X2 105.1 mm to (185.2, 113.2), turned to 90 degrees
- moved X3 100.5 mm to (185.2, 105.7), turned to 90 degrees
- moved REF** 97.2 mm to (186.2, 59.6), turned to 90 degrees
- moved X4 96.8 mm to (185.2, 98.3), turned to 90 degrees
- moved R3 96.6 mm to (173.0, 120.6), turned to 180 degrees
- moved X6 94.2 mm to (185.2, 90.9), turned to 90 degrees
- moved R5 93.5 mm to (173.0, 117.1), turned to 180 degrees
- moved X8 93.2 mm to (185.2, 68.6), turned to 90 degrees
- moved X5 92.7 mm to (185.2, 83.5), turned to 90 degrees
- moved X7 92.4 mm to (185.2, 76.0), turned to 90 degrees
- moved R8 91.1 mm to (176.5, 108.4), turned to 90 degrees
- moved R2 86.7 mm to (173.0, 108.4), turned to 90 degrees
- moved R1 82.4 mm to (169.4, 108.4), turned to 90 degrees
- moved R9 78.9 mm to (175.7, 76.6), turned to 90 degrees
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Routing:
- net Net-(D2-Pad2): track 38.6 -> 40.4 mm, vias 2 -> 0
Other:
- board size 70 x 84 mm -> 84 x 70 mm
- net class Default: via_dia 0.6 -> 0.8; via_drill 0.4 -> 0.5
- net class sinte: via_dia 0.6 -> 0.8; via_drill 0.4 -> 0.5
