File: alien.kicad_pcb (KiCad board)
At the start: 2 copper layers, 84 x 70 mm, 51 parts, among them Q1 2N3904, Q2 2N3904, Q3 2N5457, U1 LM324, X1 JD_CONN_01X01, X10 JD_CONN_01X01, X11 JD_CONN_01X01, X12 JD_CONN_01X02, X13 JD_CONN_01X02, X2 JD_CONN_01X01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

Commit message: corrección de la posición de las patas de los transistores
Parts:
- C9: value 100pF -> 0.01
- Q1, Q2: value 2N3904 -> 2N390
- moved Q1 0.19 mm to (160.9, 63.9)
- moved Q2 0.09 mm to (153.4, 63.9)
Connections:
- Q1 pad 1: Net-(Q1-Pad1) -> Net-(C7-Pad2)
- Q1 pad 2: Net-(C7-Pad2) -> Net-(Q1-Pad2)
- Q2 pad 1: GNDREF -> Net-(C8-Pad2)
- Q2 pad 2: Net-(C8-Pad2) -> GNDREF
- R10 pad 1: Net-(Q1-Pad1) -> Net-(Q1-Pad2)
- R11 pad 2: Net-(Q1-Pad1) -> Net-(Q1-Pad2)
- R12 pad 2: Net-(Q1-Pad1) -> Net-(Q1-Pad2)
- R9 pad 1: Net-(Q1-Pad1) -> Net-(Q1-Pad2)
Routing:
- net Net-(Q1-Pad2): track 0.00 -> 28.2 mm
- net Net-(Q1-Pad1): track 23.3 -> 0.00 mm
- net GNDREF: track 120.6 -> 124.7 mm
- net Net-(C8-Pad2): track 44.4 -> 45.6 mm
- net Net-(C7-Pad2): track 67.8 -> 66.7 mm, vias 3 -> 6
- net Net-(Q1-Pad3): track 34.0 -> 34.5 mm, vias 0 -> 2
- net Net-(C8-Pad1): track 67.8 -> 68.0 mm, vias 1 -> 3
- net Net-(Q3-Pad1): track 29.9 -> 30.0 mm, vias 0 -> 1
